File: Board/Board.sch (KiCad schematic (older format))
At the start: 24 parts, among them J1 Screw_Terminal_01x03, J2 Screw_Terminal_01x03, J3 Screw_Terminal_01x03, J4 Screw_Terminal_01x03, J5 Screw_Terminal_01x03, J6 Screw_Terminal_01x03, J7 Screw_Terminal_01x03, J8 Screw_Terminal_01x03, J9 Screw_Terminal_01x02, K1 SANYOU_SRD_Form_C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

Commit message: Finished PCB
Parts:
- J9: value Screw_Terminal_01x02 -> 220v; footprint TerminalBlock:TerminalBlock_Wuerth_691311400102_P7.62mm -> TerminalBlock:TerminalBlock_Altech_AK300-2_P5.00mm
Connections:
- net at U1.1 (QB): now also U3.7 (I7); no longer U3.2 (I2)
- net at U1.15 (QA): now also U3.8 (I8); no longer U3.1 (I1)
- net at U1.2 (QC): now also U3.6 (I6); no longer U3.3 (I3)
- net at U1.3 (QD): now also U3.5 (I5); no longer U3.4 (I4)
- net at U1.4 (QE): now also U3.4 (I4); no longer U3.5 (I5)
- net at U1.5 (QF): now also U3.3 (I3); no longer U3.6 (I6)
- net at U1.6 (QG): now also U3.2 (I2); no longer U3.7 (I7)
- net at U1.7 (QH): now also U3.1 (I1); no longer U3.8 (I8)
- net at J4.1 (Pin_1): now also K4.3; no longer K4.1
- net COM_RL1: now reaches J4.2 (Pin_2)
- net COM_RL1: now also K4.1; no longer K4.3
- net at J8.1 (Pin_1): now also K8.3; no longer K8.1
- net COM_RL2: now reaches J8.2 (Pin_2)
- net COM_RL2: now also K8.1; no longer K8.3
- net at J3.1 (Pin_1): now also K3.4; no longer K3.1
- net at K3.3: now also J3.3 (Pin_3); no longer J3.2 (Pin_2)
- net at J7.1 (Pin_1): now also K7.3; no longer K7.1
- net COM_RL4: now reaches J7.2 (Pin_2)
- net COM_RL4: now also K7.1; no longer K7.3
- net at J2.1 (Pin_1): now also K2.3; no longer K2.1
- net COM_RL5: now reaches J2.2 (Pin_2)
- net COM_RL5: now also K2.1; no longer K2.3
- net at J6.1 (Pin_1): now also K6.3; no longer K6.1
- net COM_RL6: now reaches J6.2 (Pin_2)
- net COM_RL6: now also K6.1; no longer K6.3
- net at J1.1 (Pin_1): now also K1.3; no longer K1.1
- net COM_RL7: now reaches J1.2 (Pin_2)
- net COM_RL7: now also K1.1; no longer K1.3
- net at J5.1 (Pin_1): now also K5.3; no longer K5.1
- net COM_RL8: now reaches J5.2 (Pin_2)
- net COM_RL8: now also K5.1; no longer K5.3
- new net COM_RL3: J3.2 (Pin_2), K3.1
Changed lines of the file:
@@
 L Transistor_Array:ULN2803A U3
 U 1 1 5DBA2C8A
-P 3000 2650
-F 0 "U3" H 3000 3217 50  0000 C CNN
-F 1 "ULN2803A" H 3000 3126 50  0000 C CNN
-F 2 "Package_DIP:DIP-18_W7.62mm_LongPads" H 3050 2000 50  0001 L CNN
-F 3 "http://www.ti.com/lit/ds/symlink/uln2803a.pdf" H 3100 2450 50  0001 C CNN
-	1    3000 2650
-	1    0    0    -1
+P 3000 2950
+F 0 "U3" H 3000 3517 50  0000 C CNN
+F 1 "ULN2803A" H 3000 3426 50  0000 C CNN
+F 2 "Package_DIP:DIP-18_W7.62mm_LongPads" H 3050 2300 50  0001 L CNN
+F 3 "http://www.ti.com/lit/ds/symlink/uln2803a.pdf" H 3100 2750 50  0001 C CNN
+	1    3000 2950
+	1    0    0    1
 $EndComp
 $Comp
 L power:GND #PWR05
 U 1 1 5DBA3F75
-P 3000 3500
-F 0 "#PWR05" H 3000 3250 50  0001 C CNN
-F 1 "GND" H 3005 3327 50  0000 C CNN
-F 2 "" H 3000 3500 50  0001 C CNN
-F 3 "" H 3000 3500 50  0001 C CNN
-	1    3000 3500
-	1    0    0    -1
-$EndComp
-Wire Wire Line
-	3000 3500 3000 3350
+P 3150 2250
+F 0 "#PWR05" H 3150 2000 50  0001 C CNN
+F 1 "GND" H 3155 2077 50  0000 C CNN
+F 2 "" H 3150 2250 50  0001 C CNN
+F 3 "" H 3150 2250 50  0001 C CNN
+	1    3150 2250
+	-1   0    0    -1
+$EndComp
+Wire Wire Line
+	3000 2100 3000 2250
 $Comp
 L ESP8266:ESP-01v090 U2
@@
 $EndComp
 NoConn ~ 2200 3350
-Wire Wire Line
-	3400 2350 3550 2350
+Text Label 3900 2450 0    50   ~ 0
+RL8
+Text Label 3900 2550 0    50   ~ 0
+RL7
+Text Label 3900 2650 0    50   ~ 0
+RL6
+Text Label 3900 2750 0    50   ~ 0
+RL5
+Text Label 3900 2850 0    50   ~ 0
+RL4
+Text Label 3900 2950 0    50   ~ 0
+RL3
+Text Label 3900 3050 0    50   ~ 0
+RL2
 Text Label 3900 3150 0    50   ~ 0
-RL8
-Text Label 3900 3050 0    50   ~ 0
-RL7
-Text Label 3900 2950 0    50   ~ 0
-RL6
-Text Label 3900 2850 0    50   ~ 0
-RL5
-Text Label 3900 2750 0    50   ~ 0
-RL4
-Text Label 3900 2650 0    50   ~ 0
-RL3
-Text Label 3900 2550 0    50   ~ 0
-RL2
-Text Label 3900 2450 0    50   ~ 0
 RL1
 Wire Wire Line
-	3900 3150 3400 3150
-Wire Wire Line
-	3400 3050 3900 3050
-Wire Wire Line
-	3900 2950 3400 2950
-Wire Wire Line
-	3400 2850 3900 2850
-Wire Wire Line
-	3900 2750 3400 2750
-Wire Wire Line
-	3400 2650 3900 2650
-Wire Wire Line
-	3900 2550 3400 2550
-Wire Wire Line
-	3400 2450 3900 2450
+	3900 2450 3400 2450
+Wire Wire Line
+	3400 2550 3900 2550
+Wire Wire Line
+	3900 2650 3400 2650
+Wire Wire Line
+	3400 2750 3900 2750
+Wire Wire Line
+	3900 2850 3400 2850
+Wire Wire Line
+	3400 2950 3900 2950
+Wire Wire Line
+	3900 3050 3400 3050
+Wire Wire Line
+	3400 3150 3900 3150
 $Comp
 L power:+5V #PWR06
 U 1 1 5DBB5436
-P 3550 2150
-F 0 "#PWR06" H 3550 2000 50  0001 C CNN
-F 1 "+5V" H 3565 2323 50  0000 C CNN
-F 2 "" H 3550 2150 50  0001 C CNN
-F 3 "" H 3550 2150 50  0001 C CNN
-	1    3550 2150
-	1    0    0    -1
-$EndComp
-Wire Wire Line
-	3550 2150 3550 2350
+P 4250 3050
+F 0 "#PWR06" H 4250 2900 50  0001 C CNN
+F 1 "+5V" H 4265 3223 50  0000 C CNN
+F 2 "" H 4250 3050 50  0001 C CNN
+F 3 "" H 4250 3050 50  0001 C CNN
+	1    4250 3050
+	-1   0    0    -1
+$EndComp
 Wire Wire Line
 	8050 1750 7950 1750
-Wire Wire Line
-	7950 1750 7950 2000
 $Comp
 L power:+5V #PWR011
@@
 	8750 1650 8750 1750
 Wire Wire Line
-	7950 2000 8750 2000
-Wire Wire Line
-	8750 1950 9000 1950
-Wire Wire Line
-	8750 2000 8750 1950
-Wire Wire Line
 	8650 1650 8750 1650
-Wire Wire Line
-	8650 1850 9000 1850
 $Comp
 L Connector:Screw_Terminal_01x03 J4
@@
 Wire Wire Line
 	9800 1750 9700 1750
-Wire Wire Line
-	9700 1750 9700 2000
 $Comp
 L power:+5V #PWR015
@@
 	10500 1650 10500 1750
 Wire Wire Line
-	9700 2000 10500 2000
-Wire Wire Line
-	10500 1950 10750 1950
-Wire Wire Line
-	10500 2000 10500 1950
-Wire Wire Line
 	10400 1650 10500 1650
-Wire Wire Line
-	10400 1850 10750 1850
 $Comp
 L Connector:Screw_Terminal_01x03 J8
@@
 Wire Wire Line
 	7950 3050 7850 3050
-Wire Wire Line
-	7850 3050 7850 3300
 $Comp
 L power:+5V #PWR010
@@
 	8650 2950 8650 3050
 Wire Wire Line
-	7850 3300 8650 3300
-Wire Wire Line
-	8650 3250 8900 3250
-Wire Wire Line
-	8650 3300 8650 3250
-Wire Wire Line
 	8550 2950 8650 2950
-Wire Wire Line
-	8550 3150 8900 3150
 $Comp
 L Connector:Screw_Terminal_01x03 J3
@@
 F 3 "~" H 9100 3150 50  0001 C CNN
 	1    9100 3150
-	1    0    0    1
+	1    0    0    -1
 $EndComp
 $Comp
@@
 Wire Wire Line
 	9700 3050 9600 3050
-Wire Wire Line
-	9600 3050 9600 3300
 $Comp
 L power:+5V #PWR014
@@
 	10400 2950 10400 3050
 Wire Wire Line
-	9600 3300 10400 3300
-Wire Wire Line
-	10400 3250 10650 3250
-Wire Wire Line
-	10400 3300 10400 3250
-Wire Wire Line
 	10300 2950 10400 2950
 Wire Wire Line
-	10300 3150 10650 3150
+	10300 3150 10350 3150
 $Comp
 L Connector:Screw_Terminal_01x03 J7
@@
 Wire Wire Line
 	7900 4250 7800 4250
-Wire Wire Line
-	7800 4250 7800 4500
 $Comp
 L power:+5V #PWR09
@@
 	8600 4150 8600 4250
 Wire Wire Line
-	7800 4500 8600 4500
-Wire Wire Line
 	8600 4450 8850 4450
 Wire Wire Line
-	8600 4500 8600 4450
-Wire Wire Line
 	8500 4150 8600 4150
-Wire Wire Line
-	8500 4350 8850 4350
 $Comp
 L Connector:Screw_Terminal_01x03 J2
@@
 Wire Wire Line
 	9650 4250 9550 4250
-Wire Wire Line
-	9550 4250 9550 4500
 $Comp
 L power:+5V #PWR013
@@
 	10350 4150 10350 4250
 Wire Wire Line
-	9550 4500 10350 4500
-Wire Wire Line
-	10350 4450 10600 4450
-Wire Wire Line
-	10350 4500 10350 4450
-Wire Wire Line
 	10250 4150 10350 4150
-Wire Wire Line
-	10250 4350 10600 4350
 $Comp
 L Connector:Screw_Terminal_01x03 J6
@@
 Wire Wire Line
 	7800 5550 7700 5550
-Wire Wire Line
-	7700 5550 7700 5800
 $Comp
 L power:+5V #PWR08
@@
 	8500 5450 8500 5550
 Wire Wire Line
-	7700 5800 8500 5800
-Wire Wire Line
-	8500 5750 8750 5750
-Wire Wire Line
-	8500 5800 8500 5750
-Wire Wire Line
 	8400 5450 8500 5450
 Wire Wire Line
-	8400 5650 8750 5650
+	8400 5650 8450 5650
 $Comp
 L Connector:Screw_Terminal_01x03 J1
@@
 Wire Wire Line
 	9550 5550 9450 5550
-Wire Wire Line
-	9450 5550 9450 5800
 $Comp
 L power:+5V #PWR012
@@
 	10250 5450 10250 5550
 Wire Wire Line
-	9450 5800 10250 5800
-Wire Wire Line
-	10250 5750 10500 5750
-Wire Wire Line
-	10250 5800 10250 5750
-Wire Wire Line
 	10150 5450 10250 5450
 Wire Wire Line
-	10150 5650 10500 5650
+	10150 5650 10200 5650
 $Comp
 L Connector:Screw_Terminal_01x03 J5
@@
 P 1400 5350
 F 0 "J9" H 1318 5025 50  0000 C CNN
-F 1 "Screw_Terminal_01x02" H 1318 5116 50  0000 C CNN
-F 2 "TerminalBlock:TerminalBlock_Wuerth_691311400102_P7.62mm" H 1400 5350 50  0001 C CNN
+F 1 "220v" H 1318 5116 50  0000 C CNN
+F 2 "TerminalBlock:TerminalBlock_Altech_AK300-2_P5.00mm" H 1400 5350 50  0001 C CNN
 F 3 "~" H 1400 5350 50  0001 C CNN
 	1    1400 5350
@@
 	2950 5900 2950 5700
 Connection ~ 2950 5700
+Wire Wire Line
+	3000 2100 3150 2100
+Wire Wire Line
+	3150 2100 3150 2250
+Wire Wire Line
+	4250 3250 4250 3050
+Wire Wire Line
+	3400 3250 4250 3250
+Wire Wire Line
+	8550 3150 8600 3150
+Wire Wire Line
+	8600 3150 8600 3250
+Wire Wire Line
+	8600 3250 8900 3250
+Text Label 7850 3050 2    50   ~ 0
+COM_RL3
+Text Label 8900 3150 2    50   ~ 0
+COM_RL3
+Text Label 7950 1750 2    50   ~ 0
+COM_RL1
+Wire Wire Line
+	8650 1850 8700 1850
+Wire Wire Line
+	8700 1850 8700 1950
+Wire Wire Line
+	8700 1950 9000 1950
+Text Label 9000 1850 2    50   ~ 0
+COM_RL1
+Text Label 9700 1750 2    50   ~ 0
+COM_RL2
+Wire Wire Line
+	10400 1850 10450 1850
+Wire Wire Line
+	10450 1850 10450 1950
+Wire Wire Line
+	10450 1950 10750 1950
+Text Label 10750 1850 2    50   ~ 0
+COM_RL2
+Text Label 9600 3050 2    50   ~ 0
+COM_RL4
+Text Label 10650 3150 2    50   ~ 0
+COM_RL4
+Wire Wire Line
+	10350 3150 10350 3250
+Wire Wire Line
+	10350 3250 10650 3250
+Text Label 7800 4250 2    50   ~ 0
+COM_RL5
+Wire Wire Line
+	8600 4350 8600 4450
+Wire Wire Line
+	8500 4350 8600 4350
+Text Label 8850 4350 2    50   ~ 0
+COM_RL5
+Text Label 9550 4250 2    50   ~ 0
+COM_RL6
+Wire Wire Line
+	10250 4350 10300 4350
+Wire Wire Line
+	10300 4450 10300 4350
+Wire Wire Line
+	10300 4450 10600 4450
+Text Label 10600 4350 2    50   ~ 0
+COM_RL6
+Text Label 9450 5550 2    50   ~ 0
+COM_RL8
+Text Label 10500 5650 2    50   ~ 0
+COM_RL8
+Wire Wire Line
+	10200 5650 10200 5750
+Wire Wire Line
+	10200 5750 10500 5750
+Text Label 7700 5550 2    50   ~ 0
+COM_RL7
+Text Label 8750 5650 2    50   ~ 0
+COM_RL7
+Wire Wire Line
+	8450 5650 8450 5750
+Wire Wire Line
+	8450 5750 8750 5750
 $EndSCHEMATC
